File: portenta_x8_carrier.kicad_sch (KiCad schematic)
At the start: 2 parts, among them J1 4049_80pos_High_Density, J2 4049_80pos_High_Density

Commit message: Started naming pins
Connections:
- net ETH_A+: now reaches J1.1 (Pin_1)
- net MIPI_DSI_D1_P: now reaches J1.10 (Pin_10)
- net ETH_C-: now reaches J1.11 (Pin_11)
- net MIPI_DSI_D1_N: now reaches J1.12 (Pin_12)
- net ETH_D+: now reaches J1.13 (Pin_13)
- net MIPI_DSI_D0_P: now reaches J1.14 (Pin_14)
- net ETH_D-: now reaches J1.15 (Pin_15)
- net MIPI_DSI_D0_N: now reaches J1.16 (Pin_16)
- net LED2_LINK: now reaches J1.17 (Pin_17)
- net MIPI_DSI_CKL_P: now reaches J1.18 (Pin_18)
- net LED2_ACT: now reaches J1.19 (Pin_19)
- net MIPI_DSI_D3_P: now reaches J1.2 (Pin_2)
- net MIPI_DSI_CKL_N: now reaches J1.20 (Pin_20)
- net VSYS_5V: now reaches J1.21 (Pin_21)
- net VSYS_5V: now also J1.32 (Pin_32), J1.41 (Pin_41), J1.48 (Pin_48), J1.53 (Pin_53), J1.64 (Pin_64)
- net GND: now reaches J1.22 (Pin_22)
- net GND: now also J1.31 (Pin_31), J1.42 (Pin_42), J1.47 (Pin_47), J1.54 (Pin_54)
- net USB1_VBUS: now reaches J1.23 (Pin_23)
- net USB2_VBUS: now reaches J1.24 (Pin_24)
- net USB1_DP: now reaches J1.25 (Pin_25)
- net USB2_DP: now reaches J1.26 (Pin_26)
- net USB1_DN: now reaches J1.27 (Pin_27)
- net USB2_DN: now reaches J1.28 (Pin_28)
- net USB1_ID: now reaches J1.29 (Pin_29)
- net ETH_A-: now reaches J1.3 (Pin_3)
- net USB2_ID: now reaches J1.30 (Pin_30)
- net UART2_TXD: now reaches J1.33 (Pin_33)
- net UART_STM32_TXD: now reaches J1.34 (Pin_34)
- net UART2_RXD: now reaches J1.35 (Pin_35)
- net UART_STM32_RXD: now reaches J1.36 (Pin_36)
- net UART2_RTS: now reaches J1.37 (Pin_37)
- net UART_STM32_RTS: now reaches J1.38 (Pin_38)
- net UART2_CTS: now reaches J1.39 (Pin_39)
- net MIPI_DSI_D3_N: now reaches J1.4 (Pin_4)
- net UART_STM32_CTS: now reaches J1.40 (Pin_40)
- net I2C2_SDA: now reaches J1.43 (Pin_43)
- net I2C3_SDA: now reaches J1.44 (Pin_44)
- net I2C2_SCL: now reaches J1.45 (Pin_45)
- net I2C3_SCL: now reaches J1.46 (Pin_46)
- net CAN1_TX: now reaches J1.49 (Pin_49)
- net ETH_B+: now reaches J1.5 (Pin_5)
- net CAN1_RX: now reaches J1.51 (Pin_51)
- net MIPI_DSI_D2_P: now reaches J1.6 (Pin_6)
- net ETH_B-: now reaches J1.7 (Pin_7)
- net MIPI_DSI_D2_N: now reaches J1.8 (Pin_8)
- net ETH_C+: now reaches J1.9 (Pin_9)
